File: Hardware/PCB/kicad/M5-Remote_v1.kicad_sch (KiCad schematic)
At the start: 35 parts, among them M5-CORE2 M5_CORE2, U1 PCA9685PW, U2 MCP23017_SS, U4 CHERRY-MX-LED

Commit message: Big rename
Parts:
- B1: symbol OSSM-M5-Remote_v1-eagle-import:JST-PH-2MM,180 -> M5-Remote_v1:JST-PH-2MM,180
- B2: symbol OSSM-M5-Remote_v1-eagle-import:JST-PH-2MM,180,reversepolarity -> M5-Remote_v1:JST-PH-2MM,180,reversepolarity
- H1, H2, H3, H4: footprint OSSM-M5-Remote_v1:mounting_hole_3.3mm -> M5-Remote_v1:mounting_hole_3.3mm
- M5-CORE2: footprint OSSM-M5-Remote_v1:M5_CORE2 -> M5-Remote_v1:M5_CORE2; symbol OSSM-M5-Remote_v1-eagle-import:M5_CORE2 -> M5-Remote_v1:M5_CORE2
- SW1, SW2, SW3, SW4: footprint OSSM-M5-Remote_v1:PEL12T4225SS1024 -> M5-Remote_v1:PEL12T4225SS1024
- U4: footprint OSSM-M5-Remote_v1:CHERRY-MX-LED -> M5-Remote_v1:CHERRY-MX-LED; symbol OSSM-M5-Remote_v1-eagle-import:CHERRY-MX-LED -> M5-Remote_v1:CHERRY-MX-LED

Commit message: Final touches for first PCB version
Parts:
- B2: value ~ -> JST-PH-2MM,180
- M5-CORE2: value M5_CORE2 -> M5Bus Header
- SW1, SW2, SW3, SW4: value ~ -> PEL12T4225SS1024
- U1: JLCPCB Rotation Offset (none) -> 90
- renumbered U4 to U3
Changed lines of the file:
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@@
 			)
 		)
-		(property "Value" "~"
+		(property "Value" "PEL12T4225SS1024"
 			(at 53.34 88.9 0)
 			(effects
@@
 			)
 		)
-		(property "Value" "~"
+		(property "Value" "PEL12T4225SS1024"
 			(at 45.72 58.42 0)
 			(effects
@@
 			)
 		)
-		(property "Value" "~"
+		(property "Value" "PEL12T4225SS1024"
 			(at 132.08 87.63 0)
 			(effects
@@
 			)
 		)
+		(property "JLCPCB Rotation Offset" "90"
+			(at 93.98 40.64 0)
+			(effects
+				(font
+					(size 1.27 1.27)
+				)
+				(hide yes)
+			)
+		)
 		(pin "6"
 		)
@@
 		(on_board yes)
 		(dnp no)
-		(property "Reference" "U4"
+		(property "Reference" "U3"
 			(at 68.326 135.636 0)
 			(effects
@@
 			(project "M5-Remote_v1"
 				(path "/34984dbd-fd6c-43b7-996b-7c11903ec195"
-					(reference "U4")
+					(reference "U3")
 					(unit 1)
 				)
@@
 			)
 		)
-		(property "Value" "~"
+		(property "Value" "PEL12T4225SS1024"
 			(at 139.7 57.15 0)
 			(effects
@@
 			)
 		)
-		(property "Value" "~"
+		(property "Value" "JST-PH-2MM,180"
 			(at 246.38 113.03 0)
 			(effects
@@
 			)
 		)
-		(property "Value" "M5_CORE2"
+		(property "Value" "M5Bus Header"
 			(at 239.014 50.8 0)
 			(effects
