File: Hardware/PCB/kicad/M5-Remote_v1.kicad_pcb (KiCad board)
At the start: 2 copper layers, 108.5 x 73.1 mm, 35 parts, among them M5-CORE2 M5_CORE2, U1 PCA9685PW, U2 MCP23017_SS, U4 Val**

Commit message: Big rename
Parts:
- H1, H2, H3, H4: footprint OSSM-M5-Remote_v1:mounting_hole_3.3mm -> M5-Remote_v1:mounting_hole_3.3mm
- M5-CORE2: footprint OSSM-M5-Remote_v1:M5_CORE2 -> M5-Remote_v1:M5_CORE2
- SW1, SW2, SW3, SW4: footprint OSSM-M5-Remote_v1:PEL12T4225SS1024 -> M5-Remote_v1:PEL12T4225SS1024
- U4: footprint OSSM-M5-Remote_v1:CHERRY-MX-LED -> M5-Remote_v1:CHERRY-MX-LED
Changed lines of the file:
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@@
 	(net 74 "/SW4_ROTA")
 	(net 75 "/CHERRY_BUTTON")
-	(footprint "OSSM-M5-Remote_v1:mounting_hole_3.3mm"
+	(footprint "M5-Remote_v1:mounting_hole_3.3mm"
 		(layer "F.Cu")
 		(at 113.5011 102.206)
@@
 			)
 		)
-		(property "Footprint" "OSSM-M5-Remote_v1:mounting_hole_3.3mm"
+		(property "Footprint" "M5-Remote_v1:mounting_hole_3.3mm"
 			(at 0 0 0)
 			(unlocked yes)
@@
 		)
 	)
-	(footprint "OSSM-M5-Remote_v1:PEL12T4225SS1024"
+	(footprint "M5-Remote_v1:PEL12T4225SS1024"
 		(layer "F.Cu")
 		(at 103.5013 109.7896)
@@
 			)
 		)
-		(property "Footprint" "OSSM-M5-Remote_v1:PEL12T4225SS1024"
+		(property "Footprint" "M5-Remote_v1:PEL12T4225SS1024"
 			(at 0 0 0)
 			(unlocked yes)
@@
 		)
 	)
-	(footprint "OSSM-M5-Remote_v1:PEL12T4225SS1024"
+	(footprint "M5-Remote_v1:PEL12T4225SS1024"
 		(layer "F.Cu")
 		(at 193.5009 109.253)
@@
 			)
 		)
-		(property "Footprint" "OSSM-M5-Remote_v1:PEL12T4225SS1024"
+		(property "Footprint" "M5-Remote_v1:PEL12T4225SS1024"
 			(at 0 0 0)
 			(unlocked yes)
@@
 		)
 	)
-	(footprint "OSSM-M5-Remote_v1:PEL12T4225SS1024"
+	(footprint "M5-Remote_v1:PEL12T4225SS1024"
 		(layer "F.Cu")
 		(at 123.5011 129.2898 180)
@@
 			)
 		)
-		(property "Footprint" "OSSM-M5-Remote_v1:PEL12T4225SS1024"
+		(property "Footprint" "M5-Remote_v1:PEL12T4225SS1024"
 			(at 0 0 180)
 			(unlocked yes)
@@
 		)
 	)
-	(footprint "OSSM-M5-Remote_v1:CHERRY-MX-LED"
+	(footprint "M5-Remote_v1:CHERRY-MX-LED"
 		(layer "F.Cu")
 		(at 148.5111 128.38)
@@
 			)
 		)
-		(property "Footprint" "OSSM-M5-Remote_v1:CHERRY-MX-LED"
+		(property "Footprint" "M5-Remote_v1:CHERRY-MX-LED"
 			(at 0 0 0)
 			(unlocked yes)
@@
 		)
 	)
-	(footprint "OSSM-M5-Remote_v1:mounting_hole_3.3mm"
+	(footprint "M5-Remote_v1:mounting_hole_3.3mm"
 		(layer "F.Cu")
 		(at 183.5011 102.206)
@@
 			)
 		)
-		(property "Footprint" "OSSM-M5-Remote_v1:mounting_hole_3.3mm"
+		(property "Footprint" "M5-Remote_v1:mounting_hole_3.3mm"
 			(at 0 0 0)
 			(unlocked yes)
@@
 		)
 	)
-	(footprint "OSSM-M5-Remote_v1:mounting_hole_3.3mm"
+	(footprint "M5-Remote_v1:mounting_hole_3.3mm"
 		(layer "F.Cu")
 		(at 162.5011 134.54)
@@
 			)
 		)
-		(property "Footprint" "OSSM-M5-Remote_v1:mounting_hole_3.3mm"
+		(property "Footprint" "M5-Remote_v1:mounting_hole_3.3mm"
 			(at 0 0 0)
 			(unlocked yes)
@@
 		)
 	)
-	(footprint "OSSM-M5-Remote_v1:PEL12T4225SS1024"
+	(footprint "M5-Remote_v1:PEL12T4225SS1024"
 		(layer "F.Cu")
 		(at 173.5009 129.29 180)
@@
 			)
 		)
-		(property "Footprint" "OSSM-M5-Remote_v1:PEL12T4225SS1024"
+		(property "Footprint" "M5-Remote_v1:PEL12T4225SS1024"
 			(at 0 0 180)
 			(unlocked yes)
@@
 		)
 	)
-	(footprint "OSSM-M5-Remote_v1:mounting_hole_3.3mm"
+	(footprint "M5-Remote_v1:mounting_hole_3.3mm"
 		(layer "F.Cu")
 		(at 134.5011 134.54)
@@
 			)
 		)
-		(property "Footprint" "OSSM-M5-Remote_v1:mounting_hole_3.3mm"
+		(property "Footprint" "M5-Remote_v1:mounting_hole_3.3mm"
 			(at 0 0 0)
 			(unlocked yes)
@@
 		)
 	)
-	(footprint "OSSM-M5-Remote_v1:M5_CORE2"
+	(footprint "M5-Remote_v1:M5_CORE2"
 		(layer "B.Cu")
 		(at 168.7711 107.32 90)
@@
 			)
 		)
-		(property "Footprint" "OSSM-M5-Remote_v1:M5_CORE2"
+		(property "Footprint" "M5-Remote_v1:M5_CORE2"
 			(at 0 0 -90)
 			(unlocked yes)

Commit message: Final touches for first PCB version
Parts:
- B2: value ~ -> JST-PH-2MM,180
- M5-CORE2: value M5_CORE2 -> M5Bus Header
- SW1, SW2, SW3, SW4: value ~ -> PEL12T4225SS1024
- U3: renamed from U4; value Val** -> CHERRY-MX-LED
Other:
- board text added: "JLCJLCJLCJLC"
Changed lines of the file:
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@@
 			)
 		)
-		(attr exclude_from_bom dnp)
+		(property ki_fp_filters "MountingHole*")
+		(sheetname "Root")
+		(sheetfile "M5-Remote_v1.kicad_sch")
+		(attr exclude_from_pos_files exclude_from_bom dnp)
 		(pad "" np_thru_hole circle
 			(at 0 0)
@@
 			)
 		)
-		(property "Value" "~"
+		(property "Value" "PEL12T4225SS1024"
 			(at 0 0 0)
 			(layer "F.SilkS")
@@
 			)
 		)
+		(sheetname "Root")
+		(sheetfile "M5-Remote_v1.kicad_sch")
 		(attr through_hole exclude_from_pos_files)
 		(fp_line
@@
 			)
 		)
-		(property "Value" "~"
+		(property "Value" "PEL12T4225SS1024"
 			(at 0 0 0)
 			(layer "F.SilkS")
@@
 			)
 		)
+		(sheetname "Root")
+		(sheetfile "M5-Remote_v1.kicad_sch")
 		(attr through_hole exclude_from_pos_files)
 		(fp_line
@@
 			)
 		)
-		(property "Value" "~"
+		(property "Value" "PEL12T4225SS1024"
 			(at 0 0 180)
 			(layer "F.SilkS")
@@
 			)
 		)
+		(sheetname "Root")
+		(sheetfile "M5-Remote_v1.kicad_sch")
 		(attr through_hole exclude_from_pos_files)
 		(fp_line
@@
 		(at 148.5111 128.38)
 		(descr "Cherry MX series keyswitch footprint with additional holes for LED")
-		(property "Reference" "U4"
+		(property "Reference" "U3"
 			(at -7.62 -7.62 0)
 			(unlocked yes)
@@
 			)
 		)
-		(property "Value" "Val**"
+		(property "Value" "CHERRY-MX-LED"
 			(at 0 0 0)
 			(unlocked yes)
@@
 			)
 		)
-		(property "JLCPCB Part Number" ""
-			(at 0 0 0)
-			(unlocked yes)
-			(layer "F.Fab")
-			(hide yes)
-			(effects
-				(font
-					(size 1 1)
-					(thickness 0.15)
-				)
-			)
-		)
 		(property "MFR Part Number" ""
 			(at 0 0 0)
@@
 			)
 		)
+		(sheetname "Root")
+		(sheetfile "M5-Remote_v1.kicad_sch")
 		(attr exclude_from_pos_files)
 		(fp_line
@@
 			)
 		)
-		(attr exclude_from_bom dnp)
+		(property ki_fp_filters "MountingHole*")
+		(sheetname "Root")
+		(sheetfile "M5-Remote_v1.kicad_sch")
+		(attr exclude_from_pos_files exclude_from_bom dnp)
 		(pad "" np_thru_hole circle
 			(at 0 0)
@@
 			)
 		)
-		(attr exclude_from_bom dnp)
+		(property ki_fp_filters "MountingHole*")
+		(sheetname "Root")
+		(sheetfile "M5-Remote_v1.kicad_sch")
+		(attr exclude_from_pos_files exclude_from_bom dnp)
 		(pad "" np_thru_hole circle
 			(at 0 0)
@@
 			)
 		)
-		(property "Value" "~"
+		(property "Value" "PEL12T4225SS1024"
 			(at 0 0 180)
 			(layer "F.SilkS")
@@
 			)
 		)
+		(sheetname "Root")
+		(sheetfile "M5-Remote_v1.kicad_sch")
 		(attr through_hole exclude_from_pos_files)
 		(fp_line
@@
 			)
 		)
-		(attr exclude_from_bom dnp)
+		(property ki_fp_filters "MountingHole*")
+		(sheetname "Root")
+		(sheetfile "M5-Remote_v1.kicad_sch")
+		(attr exclude_from_pos_files exclude_from_bom dnp)
 		(pad "" np_thru_hole circle
 			(at 0 0)
@@
 			)
 		)
+		(property ki_fp_filters "R_*")
+		(sheetname "Root")
+		(sheetfile "M5-Remote_v1.kicad_sch")
 		(attr smd)
 		(fp_line
@@
 			)
 		)
+		(property ki_fp_filters "R_*")
+		(sheetname "Root")
+		(sheetfile "M5-Remote_v1.kicad_sch")
 		(attr smd)
 		(fp_line
@@
 			)
 		)
+		(property ki_fp_filters "SSOP*5.3x10.2mm*P0.65mm*")
+		(sheetname "Root")
+		(sheetfile "M5-Remote_v1.kicad_sch")
 		(attr smd)
 		(fp_line
@@
 			)
 		)
+		(property ki_fp_filters "R_*")
+		(sheetname "Root")
+		(sheetfile "M5-Remote_v1.kicad_sch")
 		(attr smd)
 		(fp_line
@@
 			)
 		)
+		(property ki_fp_filters "R_*")
+		(sheetname "Root")
+		(sheetfile "M5-Remote_v1.kicad_sch")
 		(attr smd)
 		(fp_line
@@
 			)
 		)
+		(property ki_fp_filters "R_*")
+		(sheetname "Root")
+		(sheetfile "M5-Remote_v1.kicad_sch")
 		(attr smd)
 		(fp_line
@@
 			)
 		)
+		(property ki_fp_filters "R_*")
+		(sheetname "Root")
+		(sheetfile "M5-Remote_v1.kicad_sch")
 		(attr smd)
 		(fp_line
@@
 			)
 		)
-		(property "Value" "~"
+		(property "Value" "JST-PH-2MM,180"
 			(at 1 -7.45 90)
 			(layer "B.Fab")
@@
 			)
 		)
-		(attr through_hole)
+		(sheetname "Root")
+		(sheetfile "M5-Remote_v1.kicad_sch")
+		(attr through_hole exclude_from_pos_files)
 		(fp_line
 			(start 4.45 -6.75)
@@
 			)
 		)
-		(property "Value" "M5_CORE2"
+		(property "Value" "M5Bus Header"
 			(at 0 -4.405 -90)
 			(unlocked yes)
@@
 			)
 		)
+		(sheetname "Root")
+		(sheetfile "M5-Remote_v1.kicad_sch")
 		(attr exclude_from_pos_files)
 		(fp_line
@@
 			)
 		)
+		(property ki_fp_filters "R_*")
+		(sheetname "Root")
+		(sheetfile "M5-Remote_v1.kicad_sch")
 		(attr smd)
 		(fp_line
@@
 			)
 		)
+		(property ki_fp_filters "R_*")
+		(sheetname "Root")
+		(sheetfile "M5-Remote_v1.kicad_sch")
 		(attr smd)
 		(fp_line
@@
 			)
 		)
+		(property ki_fp_filters "R_*")
+		(sheetname "Root")
+		(sheetfile "M5-Remote_v1.kicad_sch")
 		(attr smd)
 		(fp_line
@@
 			)
 		)
+		(property ki_fp_filters "R_*")
+		(sheetname "Root")
+		(sheetfile "M5-Remote_v1.kicad_sch")
 		(attr smd)
 		(fp_line
@@
 			)
 		)
+		(property ki_fp_filters "R_*")
+		(sheetname "Root")
+		(sheetfile "M5-Remote_v1.kicad_sch")
 		(attr smd)
 		(fp_line
@@
 			)
 		)
+		(property ki_fp_filters "R_*")
+		(sheetname "Root")
+		(sheetfile "M5-Remote_v1.kicad_sch")
 		(attr smd)
 		(fp_line
@@
 			)
 		)
+		(property ki_fp_filters "R_*")
+		(sheetname "Root")
+		(sheetfile "M5-Remote_v1.kicad_sch")
 		(attr smd)
 		(fp_line
@@
 			)
 		)
-		(property "JLCPCB Part Number" ""
-			(at 0 0 90)
-			(unlocked yes)
-			(layer "B.Fab")
-			(hide yes)
-			(effects
-				(font
-					(size 1 1)
-					(thickness 0.15)
-				)
-				(justify mirror)
-			)
-		)
 		(property "MFR Part Number" ""
 			(at 0 0 90)
@@
 			)
 		)
-		(attr through_hole)
+		(sheetname "Root")
+		(sheetfile "M5-Remote_v1.kicad_sch")
+		(attr through_hole exclude_from_pos_files)
 		(fp_line
 			(start 4.45 -6.75)
@@
 			)
 		)
+		(property "JLCPCB Rotation Offset" "90"
+			(at 0 0 0)
+			(unlocked yes)
+			(layer "B.Fab")
+			(hide yes)
+			(effects
+				(font
+					(size 1 1)
+					(thickness 0.15)
+				)
+				(justify mirror)
+			)
+		)
+		(property ki_fp_filters "TSSOP*4.4x9.7mm*P0.65mm*")
+		(sheetname "Root")
+		(sheetfile "M5-Remote_v1.kicad_sch")
 		(attr smd)
 		(fp_line
@@
 			)
 		)
+		(property ki_fp_filters "R_*")
+		(sheetname "Root")
+		(sheetfile "M5-Remote_v1.kicad_sch")
 		(attr smd)
 		(fp_line
@@
 			)
 		)
+		(property ki_fp_filters "R_*")
+		(sheetname "Root")
+		(sheetfile "M5-Remote_v1.kicad_sch")
 		(attr smd)
 		(fp_line
@@
 			)
 		)
+		(property ki_fp_filters "R_*")
+		(sheetname "Root")
+		(sheetfile "M5-Remote_v1.kicad_sch")
 		(attr smd)
 		(fp_line
@@
 			)
 		)
+		(property ki_fp_filters "R_*")
+		(sheetname "Root")
+		(sheetfile "M5-Remote_v1.kicad_sch")
 		(attr smd)
 		(fp_line
@@
 			)
 		)
+		(property ki_fp_filters "C_*")
+		(sheetname "Root")
+		(sheetfile "M5-Remote_v1.kicad_sch")
 		(attr smd)
 		(fp_line
@@
 			)
 		)
+		(property ki_fp_filters "R_*")
+		(sheetname "Root")
+		(sheetfile "M5-Remote_v1.kicad_sch")
 		(attr smd)
 		(fp_line
@@
 			)
 		)
+		(property ki_fp_filters "C_*")
+		(sheetname "Root")
+		(sheetfile "M5-Remote_v1.kicad_sch")
 		(attr smd)
 		(fp_line
@@
 			)
 		)
+		(property ki_fp_filters "R_*")
+		(sheetname "Root")
+		(sheetfile "M5-Remote_v1.kicad_sch")
 		(attr smd)
 		(fp_line
@@
 		)
 	)
+	(gr_text "JLCJLCJLCJLC"
+		(at 118 102.5 0)
+		(layer "F.SilkS")
+		(effects
+			(font
+				(size 1 1)
+				(thickness 0.1)
+			)
+			(justify left bottom)
+		)
+	)

Commit message: Tiny fix
Other:
- board text removed: ""
Changed lines of the file:
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@@
-		)
-	)
-	(gr_text ""
-		(at 151.933831 74.786 0)
-		(layer "F.SilkS")
-		(effects
-			(font
-				(size 5.870956 5.870956)
-				(thickness 0.580644)
-			)
-			(justify left)
 		)
 	)
